File: hardware/apex.kicad_sch (KiCad schematic)
At the start: 23 parts, among them IC1 FE1.1S, J1 USB_C_Receptacle_USB2.0_16P, J2 USB_A, J3 USB_A, U1 USBLC6-2SC6, U2 USBLC6-2SC6, U3 USBLC6-2SC6, Y2 Crystal

Commit message: revise: apex_2
Parts:
- added H1, H2, H3, H4: MountingHole, MountingHole:MountingHole_2.2mm_M2, symbol Mechanical:MountingHole
- added TP1, TP2, TP3, TP4: TestPoint, TestPoint:TestPoint_Pad_D1.0mm, symbol Connector:TestPoint
Connections:
- net +1V8: now also TP1.1
- net +3V3: now also TP2.1
- net GND: now also TP4.1
- net VBUS: now also TP3.1
Other:
- moved on the sheet: C3, C7, C9, IC1, R3, R4, R5, U2, Y2
